File: EncoderStrainGuage.sch (KiCad schematic (older format))
At the start: 4 parts

Commit message: Updated DFFP
Parts:
- R1: symbol Device:R_Small_US -> EncoderStrainGuage-rescue:R_Small_US-Device
- U?: symbol MCU_Nordic:nRF51x22-QFxx -> EncoderStrainGuage-rescue:nRF51x22-QFxx-MCU_Nordic
Connections:
- wire segments 13 -> 12
Other:
- moved on the sheet: S?
Changed lines of the file:
@@
 EESchema Schematic File Version 4
-LIBS:EncoderStrainGuage-cache
 EELAYER 30 0
 EELAYER END
@@
 $EndDescr
 $Comp
-L EncoderBoard:StrainGuage VR?
-U 1 1 5DB7B57A
-P 7650 2100
-F 0 "VR?" H 7633 2275 50  0000 C CNN
-F 1 "StrainGuage" H 7633 2184 50  0000 C CNN
-F 2 "" H 7650 2100 50  0001 C CNN
-F 3 "" H 7650 2100 50  0001 C CNN
-	1    7650 2100
-	-1   0    0    -1
+L EncoderStrainGuage-rescue:GND-power #PWR?
+U 1 1 5DBA33BA
+P 7500 3100
+F 0 "#PWR?" H 7500 2850 50  0001 C CNN
+F 1 "GND" H 7505 2927 50  0000 C CNN
+F 2 "" H 7500 3100 50  0001 C CNN
+F 3 "" H 7500 3100 50  0001 C CNN
+	1    7500 3100
+	0    1    -1   0
 $EndComp
 $Comp
-L power:GND #PWR?
-U 1 1 5DB86977
-P 7350 2850
-F 0 "#PWR?" H 7350 2600 50  0001 C CNN
-F 1 "GND" H 7355 2677 50  0000 C CNN
-F 2 "" H 7350 2850 50  0001 C CNN
-F 3 "" H 7350 2850 50  0001 C CNN
-	1    7350 2850
-	-1   0    0    -1
-$EndComp
-Wire Wire Line
-	7250 2150 7300 2150
-$Comp
-L power:+3.3V #PWR?
-U 1 1 5DBA229F
-P 7550 2900
-F 0 "#PWR?" H 7550 2750 50  0001 C CNN
-F 1 "+3.3V" H 7565 3073 50  0000 C CNN
-F 2 "" H 7550 2900 50  0001 C CNN
-F 3 "" H 7550 2900 50  0001 C CNN
-	1    7550 2900
-	-1   0    0    -1
-$EndComp
-$Comp
-L power:GND #PWR?
-U 1 1 5DBA33BA
-P 7500 3200
-F 0 "#PWR?" H 7500 2950 50  0001 C CNN
-F 1 "GND" H 7505 3027 50  0000 C CNN
-F 2 "" H 7500 3200 50  0001 C CNN
-F 3 "" H 7500 3200 50  0001 C CNN
-	1    7500 3200
-	1    0    0    -1
-$EndComp
-Wire Wire Line
-	7350 2600 7350 2850
-$Comp
-L MCU_Nordic:nRF51x22-QFxx U?
+L EncoderStrainGuage-rescue:nRF51x22-QFxx-MCU_Nordic U?
 U 1 1 5DC073D9
 P 5500 3700
@@
 $EndComp
 $Comp
-L power:GND #PWR?
+L EncoderStrainGuage-rescue:GND-power #PWR?
 U 1 1 5DB768A9
 P 5500 5800
@@
 	1    0    0    -1
 $EndComp
-$Comp
-L power:+3.3V #PWR?
-U 1 1 5DBA0468
-P 7300 2150
-F 0 "#PWR?" H 7300 2000 50  0001 C CNN
-F 1 "+3.3V" H 7315 2323 50  0000 C CNN
-F 2 "" H 7300 2150 50  0001 C CNN
-F 3 "" H 7300 2150 50  0001 C CNN
-	1    7300 2150
-	-1   0    0    -1
-$EndComp
-$Comp
-L Device:R_Small_US R1
-U 1 1 5DB10D81
-P 7150 2150
-F 0 "R1" H 7218 2196 50  0000 L CNN
-F 1 "R" H 7218 2105 50  0000 L CNN
-F 2 "" H 7150 2150 50  0001 C CNN
-F 3 "~" H 7150 2150 50  0001 C CNN
-	1    7150 2150
-	0    -1   1    0
-$EndComp
 Wire Wire Line
 	5500 5500 5500 5800
 $Comp
-L power:+3.3V #PWR?
+L EncoderStrainGuage-rescue:+3.3V-power #PWR?
 U 1 1 5DB762A9
 P 5500 1750
@@
 Wire Wire Line
 	5500 1900 5500 1750
-Connection ~ 7300 2150
-Wire Wire Line
-	7300 2150 7350 2150
-Wire Wire Line
-	7500 3200 7750 3200
-Wire Wire Line
-	7750 2900 7550 2900
 $Comp
 L EncoderBoard:Encoder S?
 U 1 1 5DBA1183
-P 7900 3300
-F 0 "S?" V 7949 3288 50  0000 L CNN
-F 1 "Encoder" V 8040 3288 50  0000 L CNN
-F 2 "" H 7900 3300 50  0001 C CNN
-F 3 "" H 7900 3300 50  0001 C CNN
-	1    7900 3300
+P 8000 3350
+F 0 "S?" V 8049 3338 50  0000 L CNN
+F 1 "Encoder" V 8140 3338 50  0000 L CNN
+F 2 "" H 8000 3350 50  0001 C CNN
+F 3 "" H 8000 3350 50  0001 C CNN
+	1    8000 3350
 	-1   0    0    1
 $EndComp
-Wire Wire Line
-	6400 3000 7750 3000
-Wire Wire Line
-	6400 3100 7750 3100
-Wire Wire Line
-	7050 2150 6400 2150
 Wire Wire Line
 	6400 2150 6400 2200
@@
 	6400 2300 7350 2300
 Wire Wire Line
-	7350 2300 7350 2600
-Connection ~ 7350 2600
+	7050 2150 6400 2150
+Wire Wire Line
+	7300 2150 7350 2150
+Connection ~ 7300 2150
+$Comp
+L EncoderStrainGuage-rescue:R_Small_US-Device R1
+U 1 1 5DB10D81
+P 7150 2150
+F 0 "R1" H 7218 2196 50  0000 L CNN
+F 1 "R" H 7218 2105 50  0000 L CNN
+F 2 "" H 7150 2150 50  0001 C CNN
+F 3 "~" H 7150 2150 50  0001 C CNN
+	1    7150 2150
+	0    -1   1    0
+$EndComp
+$Comp
+L EncoderStrainGuage-rescue:+3.3V-power #PWR?
+U 1 1 5DBA0468
+P 7300 2150
+F 0 "#PWR?" H 7300 2000 50  0001 C CNN
+F 1 "+3.3V" H 7315 2323 50  0000 C CNN
+F 2 "" H 7300 2150 50  0001 C CNN
+F 3 "" H 7300 2150 50  0001 C CNN
+	1    7300 2150
+	-1   0    0    -1
+$EndComp
+Wire Wire Line
+	7250 2150 7300 2150
+$Comp
+L EncoderBoard:StrainGuage VR?
+U 1 1 5DB7B57A
+P 7650 2100
+F 0 "VR?" H 7633 2275 50  0000 C CNN
+F 1 "StrainGuage" H 7633 2184 50  0000 C CNN
+F 2 "" H 7650 2100 50  0001 C CNN
+F 3 "" H 7650 2100 50  0001 C CNN
+	1    7650 2100
+	-1   0    0    -1
+$EndComp
+Wire Wire Line
+	7350 2300 7350 2550
+$Comp
+L EncoderStrainGuage-rescue:GND-power #PWR?
+U 1 1 5DB86977
+P 7350 2550
+F 0 "#PWR?" H 7350 2300 50  0001 C CNN
+F 1 "GND" H 7355 2377 50  0000 C CNN
+F 2 "" H 7350 2550 50  0001 C CNN
+F 3 "" H 7350 2550 50  0001 C CNN
+	1    7350 2550
+	-1   0    0    -1
+$EndComp
+Connection ~ 7350 2550
+Wire Wire Line
+	7350 2550 7350 2600
+Wire Wire Line
+	7850 3000 6400 3000
+Wire Wire Line
+	6400 3200 7850 3200
+Wire Wire Line
+	7850 3100 7500 3100
 $EndSCHEMATC

Commit message: Add my schematic to the repo
Parts:
- added AE?: Antenna, MASA_Library:ANTC3216X140N, symbol Device:Antenna
- added BT?: Battery_Cell, 1072TR:1072TR, symbol Device:Battery_Cell
- added C? (x2): 310 pF, Capacitor_SMD:C_0603_1608Metric, symbol Device:C
- added C?: 100nF, Capacitor_SMD:C_0201_0603Metric, symbol Device:C
- added C? (x2): 15pF, Capacitor_SMD:C_0201_0603Metric, symbol Device:C
- added C? (x2): 100n, Capacitor_SMD:C_0201_0603Metric, symbol Device:C
- added C? (x4): ?, Capacitor_SMD:C_0603_1608Metric, symbol Device:C
- added D?: D_Photo, Diode_SMD:D_0603_1608Metric, symbol Device:D_Photo
- added FL?: LFB182G45BG2D280, LFB182G45BG2D280:LFB182G45BG5D920_1, symbol LFB182G45BG2D280:LFB182G45BG2D280
- added J?: Conn_01x05, Connector_PinHeader_2.54mm:PinHeader_1x05_P2.54mm_Vertical, symbol Connector_Generic:Conn_01x05
- added J? (x2): MM8130-2600RA2, MURATA_MM8130-2600RA2, symbol MM8130-2600RA2:MM8130-2600RA2
- added L?: 1.58 uH, Inductor_SMD:L_0603_1608Metric_Pad1.05x0.95mm_HandSolder, symbol Device:L
- added L? (x2): ?, Inductor_SMD:L_0603_1608Metric_Pad1.05x0.95mm_HandSolder, symbol Device:L
- added Q?: NX3020NAK,215, NX3020NAK_215:SOT95P230X110-3N, symbol NX3020NAK_215:NX3020NAK,215
- added R?: 9 MOmhs, Resistor_SMD:R_0603_1608Metric, symbol Device:R
- added R?: 10kOhm, Resistor_SMD:R_0603_1608Metric, symbol Device:R
- added R?: 56 kohm, Resistor_SMD:R_0201_0603Metric, symbol pspice:R
- added R? (x2): 100, Resistor_SMD:R_0201_0603Metric, symbol Device:R
- added R?: 10k, Resistor_SMD:R_0201_0603Metric, symbol Device:R
- added U?: OPAMP, MCP6001T-I_OT:SOT95P270X145-5N, symbol Simulation_SPICE:OPAMP
- added U?: PIC16LF88-I_SO, PIC16LF88-I_SO:SOIC127P1030X265-18N, symbol 2019-12-16_16-51-55:PIC16LF88-I_SO
- added U?: CC2500RGP, CC2500RGP:QFN50P400X400X90-21N, symbol 2019-12-22_15-43-08:CC2500RGP
- added Y?: Crystal 26-27 MHZ, ECS-260-10-36B-CKY-TR:ECS240836QAESTR, symbol Device:Crystal
Connections:
- net labels added: +5V, MCLR, PDC, PGC, PGD
- wire segments 12 -> 109
Other:
- moved on the sheet: R1, S?, U?

Commit message: finished the ant module of the schematic
Parts:
- removed C?: 100nF, Capacitor_SMD:C_0201_0603Metric, symbol Device:C
- removed C? (x2): 15pF, Capacitor_SMD:C_0201_0603Metric, symbol Device:C
- removed Q?: NX3020NAK,215, NX3020NAK_215:SOT95P230X110-3N, symbol NX3020NAK_215:NX3020NAK,215
- removed R?: 56 kohm, Resistor_SMD:R_0201_0603Metric, symbol pspice:R
- removed U?: CC2500RGP, CC2500RGP:QFN50P400X400X90-21N, symbol 2019-12-22_15-43-08:CC2500RGP
- removed Y?: Crystal 26-27 MHZ, ECS-260-10-36B-CKY-TR:ECS240836QAESTR, symbol Device:Crystal
- added C?: 1m, symbol Device:C
- added C?: 100n, symbol Device:C
- added C? (x4): 100nf, symbol Device:C
- added C?: 220pf, symbol Device:C
- added C?: 2.4 pf, symbol Device:C
- added C?: 1u, symbol Device:C
- added C? (x2): 15p, symbol Device:C
- added C? (x2): C, symbol Device:C
- added R?: 56k, symbol Device:R
- added R? (x3): 0, symbol Device:R
- added R? (x3): 100k, symbol Device:R
- added U?: CC2570RHAT, RHA40_4P5X4P5, symbol 2020-01-19_20-39-15:CC2570RHAT
- added Y?: Crystal, symbol Device:Crystal
- added Y?: Crystal_GND24, symbol Device:Crystal_GND24
- C9: renamed from C?; value ? -> 1.5 pf
- L2: renamed from L?; value ? -> 3.9 nH
- R1: footprint (none) -> Resistor_SMD:R_0201_0603Metric
- gave numbers to parts that had none: 26
Connections:
- net labels added: PSout, RFneg, RFpos, RTS, Reset, Sleep, Suspend, UARTrx, UARTtx, XOSC1, XOSC2, XOSC32K1, XOSC32K2
- net labels removed: PDC
- wire segments 109 -> 111
Other:
- moved on the sheet: C9, L2, NP1, NP2, NP3, NP4, R1, S1, U4

Commit message: fixed ant module to correct one, fixed wiring to ant module,  and added temp sensor
Parts:
- added IC?: LM60CIM3_NOPB, SOT95P237X112-3N, symbol LM60CIM3_NOPB:LM60CIM3_NOPB
- C10, C13, C14, C15, C16, C17, C18, C5, C6, C7, C8: renamed from C?; footprint (none) -> Capacitor_SMD:C_0201_0603Metric
- C11, C12: renamed from C?; value C -> 12p; footprint (none) -> Capacitor_SMD:C_0201_0603Metric
- R10, R11, R12, R13, R7, R8, R9: renamed from R?; footprint (none) -> Resistor_SMD:R_0201_0603Metric
- U3: renamed from U?; footprint RHA40_4P5X4P5 -> QFN40P500X500X90-41N:QFN40P500X500X90-41N
- Y1: renamed from Y?; footprint (none) -> CM7V-T1A_32.768KHZ_12.5PF_20PP:CM7VT1A32768KHZ125PF20PPMTAQC
- gave numbers to parts that had none: 1
Connections:
- net labels added: TempOut
- wire segments 111 -> 118
Other:
- moved on the sheet: C1, C13, C18, C2, C3, C4, C8, L1, R2, R3, R4, R5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

Commit message: added str. guage and encoder to PIC
Parts:
- removed U4: nRF51x22-QFxx, Package_DFN_QFN:QFN-48-1EP_6x6mm_P0.4mm_EP4.6x4.6mm, symbol EncoderStrainGuage-rescue:nRF51x22-QFxx-MCU_Nordic
- AE1: symbol Device:Antenna -> EncoderStrainGuage-rescue:Antenna-Device
- BT1: symbol Device:Battery_Cell -> EncoderStrainGuage-rescue:Battery_Cell-Device
- C1, C10, C11, C12, C13, C14, C15, C16, C17, C18, C2, C3, C4, C5, C6, C7, C8, C9, NP1, NP2, NP4: symbol Device:C -> EncoderStrainGuage-rescue:C-Device
- D1: symbol Device:D_Photo -> EncoderStrainGuage-rescue:D_Photo-Device
- FL1: symbol LFB182G45BG2D280:LFB182G45BG2D280 -> EncoderStrainGuage-rescue:LFB182G45BG2D280-LFB182G45BG2D280
- IC?: symbol LM60CIM3_NOPB:LM60CIM3_NOPB -> EncoderStrainGuage-rescue:LM60CIM3_NOPB-LM60CIM3_NOPB
- J1: symbol Connector_Generic:Conn_01x05 -> EncoderStrainGuage-rescue:Conn_01x05-Connector_Generic
- J2, J3: symbol MM8130-2600RA2:MM8130-2600RA2 -> EncoderStrainGuage-rescue:MM8130-2600RA2-MM8130-2600RA2
- L1, L2, NP3: symbol Device:L -> EncoderStrainGuage-rescue:L-Device
- R10, R11, R12, R13, R2, R3, R4, R5, R6, R7, R8, R9: symbol Device:R -> EncoderStrainGuage-rescue:R-Device
- U1: symbol 2019-12-16_16-51-55:PIC16LF88-I_SO -> EncoderStrainGuage-rescue:PIC16LF88-I_SO-2019-12-16_16-51-55
- U2: symbol Simulation_SPICE:OPAMP -> EncoderStrainGuage-rescue:OPAMP-Simulation_SPICE
- U3: symbol 2020-01-19_20-39-15:CC2570RHAT -> EncoderStrainGuage-rescue:CC2570RHAT-2020-01-19_20-39-15
- VR1: symbol EncoderBoard:StrainGuage -> EncoderStrainGuage-rescue:StrainGuage-EncoderBoard
- Y1: symbol Device:Crystal_GND24 -> EncoderStrainGuage-rescue:Crystal_GND24-Device
- Y2: symbol Device:Crystal -> EncoderStrainGuage-rescue:Crystal-Device
Connections:
- net labels added: +3.3V-power, EncA, EncB, Str1, Str2
- wire segments 118 -> 116
Other:
- moved on the sheet: C1, R1, R2, S1

Commit message: Gamers added filters
Parts:
- removed S1: Encoder, symbol EncoderBoard:Encoder
- added C19, C20: 310 pF, Capacitor_SMD:C_0603_1608Metric, symbol EncoderStrainGuage-rescue:C-Device
- added J4: Rotary Encoder, Connector_PinHeader_2.54mm:PinHeader_1x03_P2.54mm_Vertical, symbol Connector:Conn_01x03_Male
- added R14: 10k, Resistor_SMD:R_0603_1608Metric, symbol Device:R
- added R15, R16, R17: 10K, Resistor_SMD:R_0603_1608Metric, symbol Device:R
- C1, C10, C11, C12, C13, C14, C15, C16, C17, C18, C4, C5, C6, C7, C8: footprint Capacitor_SMD:C_0201_0603Metric -> Capacitor_SMD:C_0603_1608Metric
- IC1: renamed from IC?; footprint SOT95P237X112-3N -> LM60CIM3_NOPB:SOT95P237X112-3N
- R1, R10, R11, R12, R13, R2, R5, R6, R7, R8, R9: footprint Resistor_SMD:R_0201_0603Metric -> Resistor_SMD:R_0603_1608Metric
- VR1: footprint (none) -> Connector_PinHeader_2.54mm:PinHeader_1x02_P2.54mm_Vertical
- Y1: footprint CM7V-T1A_32.768KHZ_12.5PF_20PP:CM7VT1A32768KHZ125PF20PPMTAQC -> FA-128_32.0000MF20X-K3:FA128
- Y2: footprint (none) -> CM7V-T1A_32.768KHZ_12.5PF_20PP:CM7VT1A32768KHZ125PF20PPMTAQC
Connections:
- net +3V3: now also C19.2, C20.1, J4.2 (Pin_2), R14.1, R15.2; no longer U1.10 (RB4/SCK/SCL), U1.9 (RB3/PGM/CCP1)
- new net: R15.1, R16.1
- new net: R14.2, R17.2
- new net EncA: C19.1, J4.3 (Pin_3), R16.2, U1.9 (RB3/PGM/CCP1)
- new net EncB: C20.2, J4.1 (Pin_1), R17.1, U1.10 (RB4/SCK/SCL)

Commit message: first route on the board
Parts:
- removed BT1: Battery_Cell, 1072TR:1072TR, symbol EncoderStrainGuage-rescue:Battery_Cell-Device
- removed C19, C20: 310 pF, Capacitor_SMD:C_0603_1608Metric, symbol EncoderStrainGuage-rescue:C-Device
- removed D1: D_Photo, Diode_SMD:D_0603_1608Metric, symbol EncoderStrainGuage-rescue:D_Photo-Device
- removed R14: 10k, Resistor_SMD:R_0603_1608Metric, symbol Device:R
- removed R15, R16, R17: 10K, Resistor_SMD:R_0603_1608Metric, symbol Device:R
- added C19: 22pF, Capacitor_SMD:C_0603_1608Metric, symbol Device:C
- added C20: 10uF, Capacitor_SMD:C_0603_1608Metric, symbol Device:C
- added J5, J6: Conn_01x02_Male, Connector_PinHeader_1.00mm:PinHeader_1x02_P1.00mm_Vertical, symbol Connector:Conn_01x02_Male
- added L3: 2.2uH, Inductor_SMD:L_0603_1608Metric_Pad1.05x0.95mm_HandSolder, symbol Device:L
- added R14: 100k, Resistor_SMD:R_0603_1608Metric, symbol Device:R_US
- added R15: 450k, Resistor_SMD:R_0603_1608Metric, symbol Device:R_US
- added U4: AP3428KTTR, Package_TO_SOT_SMD:SOT-23-5, symbol AP3428KTTR:AP3428KTTR
- J4: footprint Connector_PinHeader_2.54mm:PinHeader_1x03_P2.54mm_Vertical -> Connector_PinHeader_1.00mm:PinHeader_1x02_P1.00mm_Vertical
- VR1: footprint Connector_PinHeader_2.54mm:PinHeader_1x02_P2.54mm_Vertical -> Connector_PinHeader_1.00mm:PinHeader_1x02_P1.00mm_Vertical
Connections:
- net +5V is gone; now on net +3V3: U2.4 (V+)
- net +3V3: now also J4.3 (Pin_3), R1.1, C19.1, C20.1, R14.2, R15.1, U4.5 (FB); no longer C1.2, C10.1, C11.1, C12.2, C13.2, C14.1, C15.2, C16.1, C17.1, C18.1, C2.2, C3.2, C4.2, C5.2, C6.2, C7.1, C8.2, C9.2, FL1.2 (GND_1), FL1.5 (GND_2), FL1.6 (GND_3), IC1.3 (GND), J1.3 (Pin_3), J2.GND1 (GND), J2.GND2 (GND), J2.GND3 (GND), J2.GND4 (GND), J3.GND1 (GND), J3.GND2 (GND), J3.GND3 (GND), J3.GND4 (GND), J4.2 (Pin_2), NP1.2, NP2.2, NP4.2, R1.2, R11.2, R13.1, R4.1, R7.2, R9.2, U1.17 (RA0/AN0), U1.5 (VSS), U2.2 (-), U2.5 (V-), U3.1 (GND), U3.13 (GND), U3.17 (GND), U3.2 (GND), U3.3 (GND), U3.35 (GND), U3.37 (GND), U3.38 (GND), U3.4 (GND), U3.41 (EPAD), VR1.1, VR1.2, Y1.2, Y1.4
- net RFneg: now also FL1.4 (BALANCE_PORT_2); no longer FL1.3 (BALANCE_PORT_1)
- net RFpos: now also FL1.3 (BALANCE_PORT_1); no longer FL1.4 (BALANCE_PORT_2)
- net Str1: now also R1.2, VR1.1; no longer R1.1
- net at R3.2, U2.1 (+): now also J6.1 (Pin_1)
- net PotOut: now reaches U1.1 (RA2/AN2/CVREF/VREF-)
- net PotOut: now also J4.2 (Pin_2)
- net EncA: no longer names the net of U1.9 (RB3/PGM/CCP1)
- net EncA: no longer J4.3 (Pin_3)
- net EncB: no longer names the net of U1.10 (RB4/SCK/SCL)
- net EncB: no longer J4.1 (Pin_1)
- new net: L3.1, U4.3 (LX)
- new net: C19.2, L3.2, R15.2
- new net GND: C1.2, C10.1, C11.1, C12.2, C13.2, C14.1, C15.2, C16.1, C17.1, C18.1, C2.2, C20.2, C3.2, C4.2, C5.2, C6.2, C7.1, C8.2, C9.2, FL1.2 (GND_1), FL1.5 (GND_2), FL1.6 (GND_3), IC1.3 (GND), J1.3 (Pin_3), J2.GND1 (GND), J2.GND2 (GND), J2.GND3 (GND), J2.GND4 (GND), J3.GND1 (GND), J3.GND2 (GND), J3.GND3 (GND), J3.GND4 (GND), J4.1 (Pin_1), J5.2 (Pin_2), J6.2 (Pin_2), NP1.2, NP2.2, NP4.2, R11.2, R13.1, R14.1, R4.1, R7.2, R9.2, U1.5 (VSS), U2.2 (-), U2.5 (V-), U3.1 (GND), U3.13 (GND), U3.17 (GND), U3.2 (GND), U3.3 (GND), U3.35 (GND), U3.37 (GND), U3.38 (GND), U3.4 (GND), U3.41 (EPAD), U4.2 (GND), VR1.2, Y1.2, Y1.4
- new net Vin: J5.1 (Pin_1), U4.1 (En), U4.4 (Vin)

Commit message: Fixed filter
Parts:
- C2: value 310 pF -> 1nF
- C3: value 310 pF -> 2.2uF
- L1: value 1.58 uH -> 2.2uH
Changed lines of the file:
@@
 P 7800 6550
 F 0 "L1" V 7619 6550 50  0000 C CNN
-F 1 "1.58 uH" V 7710 6550 35  0000 C CNN
+F 1 "2.2uH" V 7710 6550 35  0000 C CNN
 F 2 "Inductor_SMD:L_0603_1608Metric_Pad1.05x0.95mm_HandSolder" H 7800 6550 50  0001 C CNN
 F 3 "~" H 7800 6550 50  0001 C CNN
@@
 P 7500 6900
 F 0 "C2" H 7615 6813 50  0000 L CNN
-F 1 "310 pF" H 7615 6734 35  0000 L CNN
+F 1 "1nF" H 7615 6734 35  0000 L CNN
 F 2 "Capacitor_SMD:C_0603_1608Metric" H 7538 6750 50  0001 C CNN
 F 3 "~" H 7500 6900 50  0001 C CNN
@@
 P 8200 6900
 F 0 "C3" H 8315 6813 50  0000 L CNN
-F 1 "310 pF" H 8206 6734 35  0000 L CNN
+F 1 "2.2uF" H 8206 6734 35  0000 L CNN
 F 2 "Capacitor_SMD:C_0603_1608Metric" H 8238 6750 50  0001 C CNN
 F 3 "~" H 8200 6900 50  0001 C CNN
@@
 	5600 6450 5600 6950
 $Comp
-L power:+3.3V #PWR?
+L power:+3.3V #PWR0111
 U 1 1 5E5B2101
 P 6500 6250
-F 0 "#PWR?" H 6500 6100 50  0001 C CNN
+F 0 "#PWR0111" H 6500 6100 50  0001 C CNN
 F 1 "+3.3V" H 6515 6423 50  0000 C CNN
 F 2 "" H 6500 6250 50  0001 C CNN
